File: _autosave-AS3320-VCF.kicad_pcb (KiCad board)
At the start: 2 copper layers, 67.2 x 91.3 mm, 41 parts, among them J1 AUDIO INPUT, J2 RESONANCE CNTL. INPUT, J3 FREQ CNTL. INPUT, J4 AUDIO OUTPUT, U1 AS3320

Commit message: Refactor to use switched audio jacks.
Parts:
- removed J1: AUDIO INPUT, SeattleSynths:Jack_3.5mm_QingPu_WQP-PJ398SM_Vertical_CircularHoles
- added J5: SIGNAL_INPUT, SeattleSynths:Jack_3.5mm_QingPu_WQP-PJ398SM_Vertical_CircularHoles, B.Cu at (186.1, 109.9)
Connections:
- J2 pad T: (no net) -> /RESONANCE_CTRL_INPUT
- R8 pad 2: Net-(R8-Pad2) -> /RESONANCE_CTRL_INPUT
- RV1 pad 2: Net-(R8-Pad2) -> /RESONANCE_CTRL_INPUT
- TP1 pad 1: Net-(R8-Pad2) -> /RESONANCE_CTRL_INPUT
Routing:
- net Net-(R8-Pad2): track 103.3 -> 0.00 mm
- net /RESONANCE_CTRL_INPUT: track 0.00 -> 103.3 mm
