File: _autosave-AS3320-VCF.kicad_pcb (KiCad board)
At the start: 2 copper layers, 71.2 x 131.1 mm, 48 parts, among them J1 SIGNAL_INPUT, J2 RESONANCE_CTRL_INPUT, J3 FREQ_CTRL_INPUT, J4 SIGNAL_OUTPUT, J5 EURO_PWR_2x5, U1 AS3320

Commit message: Refactor
Parts:
- J5: value EURO_PWR_2x5 -> -----
Changed lines of the file:
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@@
       (drillshape 0)
       (scaleselection 1)
-      (outputdirectory "Gerber/"))
+      (outputdirectory "Gerbers/"))
   )
   (net 0 "")
@@
       (effects (font (size 1 1) (thickness 0.15)))
     )
-    (fp_text value EURO_PWR_2x5 (at 1.27 12.49) (layer F.SilkS)
-      (effects (font (size 1 1) (thickness 0.15)))
-    )
+    (fp_text value ----- (at 1.27 12.49) (layer F.SilkS)
+      (effects (font (size 1 1) (thickness 0.15)))
+    )
