File: AS3320-VCF.sch (KiCad schematic (older format))
At the start: 41 parts, among them J1 SIGNAL_INPUT, J2 RESONANCE_CTRL_INPUT, J3 FREQ_CTRL_INPUT, J4 SIGNAL_OUTPUT, U1 AS3320

Commit message: Refactor
Parts:
- added C6, C7: 10uF, symbol Device:C
- added J?: EURO_PWR_2x5, symbol Seattle_Synths:EURO_PWR_2x5
- TP3: value GND -> -12V
- TP4: value -12V -> GND
Connections:
- net +12V: now also C7.2, J?.1 (+12V), J?.2 (+12V)
- net -12V: now also TP3.1, C6.1, J?.10 (-12V), J?.9 (-12V); no longer TP4.1
- net GND: now also TP4.1, C6.2, C7.1, J?.3 (GND), J?.4 (GND), J?.5 (GND), J?.6 (GND), J?.7 (GND), J?.8 (GND); no longer TP3.1
Other:
- moved on the sheet: C1, C2, C3, C4, C5, D1, J1, J2, J3, J4, R1, R10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

Commit message: Refactor
Parts:
- gave numbers to parts that had none: 1
Connections:
- no-connect marks 0 -> 4
Changed lines of the file:
@@
 	9450 5200 9450 5350
 $Comp
-L Seattle_Synths:EURO_PWR_2x5 J?
+L Seattle_Synths:EURO_PWR_2x5 J5
 U 1 1 5FD28C75
 P 7400 5500
-F 0 "J?" H 7400 5947 60  0000 C CNN
+F 0 "J5" H 7400 5947 60  0000 C CNN
 F 1 "EURO_PWR_2x5" H 7400 5841 60  0000 C CNN
 F 2 "" H 7400 5500 60  0000 C CNN
@@
 $EndComp
 $Comp
-L power:-12V #PWR?
+L power:-12V #PWR0101
 U 1 1 5FD3944D
 P 7850 5700
-F 0 "#PWR?" H 7850 5800 50  0001 C CNN
+F 0 "#PWR0101" H 7850 5800 50  0001 C CNN
 F 1 "-12V" V 7850 5900 50  0000 C CNN
 F 2 "" H 7850 5700 50  0001 C CNN
@@
 $EndComp
 $Comp
-L power:-12V #PWR?
+L power:-12V #PWR0102
 U 1 1 5FD39A94
 P 6950 5700
-F 0 "#PWR?" H 6950 5800 50  0001 C CNN
+F 0 "#PWR0102" H 6950 5800 50  0001 C CNN
 F 1 "-12V" V 6950 5900 50  0000 C CNN
 F 2 "" H 6950 5700 50  0001 C CNN
@@
 $EndComp
 $Comp
-L power:+12V #PWR?
+L power:+12V #PWR0103
 U 1 1 5FD3A121
 P 7850 5300
-F 0 "#PWR?" H 7850 5150 50  0001 C CNN
+F 0 "#PWR0103" H 7850 5150 50  0001 C CNN
 F 1 "+12V" V 7850 5500 50  0000 C CNN
 F 2 "" H 7850 5300 50  0001 C CNN
@@
 $EndComp
 $Comp
-L power:+12V #PWR?
+L power:+12V #PWR0104
 U 1 1 5FD3A8F0
 P 6950 5300
-F 0 "#PWR?" H 6950 5150 50  0001 C CNN
+F 0 "#PWR0104" H 6950 5150 50  0001 C CNN
 F 1 "+12V" V 6950 5500 50  0000 C CNN
 F 2 "" H 6950 5300 50  0001 C CNN
@@
 $EndComp
 $Comp
-L power:GND #PWR?
+L power:GND #PWR0105
 U 1 1 5FD3AEB7
 P 7850 5400
-F 0 "#PWR?" H 7850 5150 50  0001 C CNN
+F 0 "#PWR0105" H 7850 5150 50  0001 C CNN
 F 1 "GND" V 7855 5227 50  0000 C CNN
 F 2 "" H 7850 5400 50  0001 C CNN
@@
 $EndComp
 $Comp
-L power:GND #PWR?
+L power:GND #PWR0106
 U 1 1 5FD3B3CF
 P 7850 5500
-F 0 "#PWR?" H 7850 5250 50  0001 C CNN
+F 0 "#PWR0106" H 7850 5250 50  0001 C CNN
 F 1 "GND" V 7855 5327 50  0000 C CNN
 F 2 "" H 7850 5500 50  0001 C CNN
@@
 $EndComp
 $Comp
-L power:GND #PWR?
+L power:GND #PWR0107
 U 1 1 5FD3B7D4
 P 7850 5600
-F 0 "#PWR?" H 7850 5350 50  0001 C CNN
+F 0 "#PWR0107" H 7850 5350 50  0001 C CNN
 F 1 "GND" V 7855 5427 50  0000 C CNN
 F 2 "" H 7850 5600 50  0001 C CNN
@@
 $EndComp
 $Comp
-L power:GND #PWR?
+L power:GND #PWR0108
 U 1 1 5FD3C716
 P 6950 5400
-F 0 "#PWR?" H 6950 5150 50  0001 C CNN
+F 0 "#PWR0108" H 6950 5150 50  0001 C CNN
 F 1 "GND" V 6955 5227 50  0000 C CNN
 F 2 "" H 6950 5400 50  0001 C CNN
@@
 $EndComp
 $Comp
-L power:GND #PWR?
+L power:GND #PWR0109
 U 1 1 5FD3CD0C
 P 6950 5500
-F 0 "#PWR?" H 6950 5250 50  0001 C CNN
+F 0 "#PWR0109" H 6950 5250 50  0001 C CNN
 F 1 "GND" V 6955 5327 50  0000 C CNN
 F 2 "" H 6950 5500 50  0001 C CNN
@@
 $EndComp
 $Comp
-L power:GND #PWR?
+L power:GND #PWR0110
 U 1 1 5FD3D018
 P 6950 5600
-F 0 "#PWR?" H 6950 5350 50  0001 C CNN
+F 0 "#PWR0110" H 6950 5350 50  0001 C CNN
 F 1 "GND" V 6955 5427 50  0000 C CNN
 F 2 "" H 6950 5600 50  0001 C CNN
@@
 	0    1    1    0
 $EndComp
+NoConn ~ 9350 2600
+NoConn ~ 1900 5350
+NoConn ~ 1900 4700
+NoConn ~ 1500 2650
 $EndSCHEMATC

Commit message: Refactor
Parts:
- C1, C2, C3, C4: footprint SeattleSynths:C_Disc_D7.5mm_W2.5mm_P5.00mm -> Seattle_Synths:C_Disc_D7.5mm_W2.5mm_P5.00mm
- C5: footprint SeattleSynths:CP_Radial_D5.0mm_P2.50mm -> Seattle_Synths:CP_Radial_D5.0mm_P2.50mm
- C6, C7: footprint (none) -> Seattle_Synths:CP_Radial_D5.0mm_P2.50mm
- D1: footprint SeattleSynths:LED_D5.0mm -> Seattle_Synths:LED_D5.0mm
- J1, J2, J3, J4: footprint SeattleSynths:Jack_3.5mm_QingPu_WQP-PJ398SM_Vertical_CircularHoles -> Seattle_Synths:Jack_3.5mm_QingPu_WQP-PJ398SM_Vertical_CircularHoles
- J5: footprint (none) -> Seattle_Synths:PinHeader_2x05_P2.54mm_Vertical
- R1, R10, R11, R12, R13, R14, R15, R16, R17, R18, R19, R2, R20, R21, R3, R4, R5, R6, R7, R8, R9: footprint SeattleSynths:R_Axial_DIN0207_L6.3mm_D2.5mm_P10.16mm_Horizontal -> Seattle_Synths:R_Axial_DIN0207_L6.3mm_D2.5mm_P10.16mm_Horizontal
- RV1, RV2: footprint SeattleSynths:Potentiometer_Alpha_RD901F-40-00D_Single_Vertical -> Seattle_Synths:Potentiometer_Alpha_RD901F-40-00D_Single_Vertical
- TP1, TP2, TP3, TP4, TP5, TP6, TP7: footprint SeattleSynths:TestPoint_Pad_4.0x4.0mm -> Seattle_Synths:TestPoint_Pad_4.0x4.0mm
- U1: footprint SeattleSynths:DIP-18_W7.62mm -> Seattle_Synths:DIP-18_W7.62mm_Socket
