File: AS3320-VCF.sch (KiCad schematic (older format))
At the start: 44 parts, among them J1 SIGNAL_INPUT, J2 RESONANCE_CTRL_INPUT, J3 FREQ_CTRL_INPUT, J4 SIGNAL_OUTPUT, J5 EURO_PWR_2x5, U1 AS3320

Commit message: Rev. 1
Parts:
- C6, C7: value 10uF -> 10µF
Changed lines of the file:
@@
 P 8950 5650
 F 0 "C6" V 8698 5650 50  0000 C CNN
-F 1 "10uF" V 8789 5650 50  0000 C CNN
+F 1 "10µF" V 8789 5650 50  0000 C CNN
 F 2 "Seattle_Synths:CP_Radial_D5.0mm_P2.50mm" H 8988 5500 50  0001 C CNN
 F 3 "~" H 8950 5650 50  0001 C CNN
@@
 P 9950 5650
 F 0 "C7" V 9698 5650 50  0000 C CNN
-F 1 "10uF" V 9789 5650 50  0000 C CNN
+F 1 "10µF" V 9789 5650 50  0000 C CNN
 F 2 "Seattle_Synths:CP_Radial_D5.0mm_P2.50mm" H 9988 5500 50  0001 C CNN
 F 3 "~" H 9950 5650 50  0001 C CNN

Commit message: Schematic Rev. 2
Parts:
- removed C2: 300pF, Seattle_Synths:C_Disc_D7.5mm_W2.5mm_P5.00mm, symbol Device:C
- removed C5: 1µF, Seattle_Synths:CP_Radial_D5.0mm_P2.50mm, symbol Device:C_Polarized
- removed C6: 10µF, Seattle_Synths:CP_Radial_D5.0mm_P2.50mm, symbol Device:C
- removed J1: SIGNAL_INPUT, Seattle_Synths:Jack_3.5mm_QingPu_WQP-PJ398SM_Vertical_CircularHoles, symbol Connector:AudioJack2_SwitchT
- removed J2: RESONANCE_CTRL_INPUT, Seattle_Synths:Jack_3.5mm_QingPu_WQP-PJ398SM_Vertical_CircularHoles, symbol Connector:AudioJack2_SwitchT
- removed J3: FREQ_CTRL_INPUT, Seattle_Synths:Jack_3.5mm_QingPu_WQP-PJ398SM_Vertical_CircularHoles, symbol Connector:AudioJack2_SwitchT
- removed J4: SIGNAL_OUTPUT, Seattle_Synths:Jack_3.5mm_QingPu_WQP-PJ398SM_Vertical_CircularHoles, symbol Connector:AudioJack2_SwitchT
- removed R1: 330R, Seattle_Synths:R_Axial_DIN0207_L6.3mm_D2.5mm_P10.16mm_Horizontal, symbol Device:R
- removed R10, R19: 1K8, Seattle_Synths:R_Axial_DIN0207_L6.3mm_D2.5mm_P10.16mm_Horizontal, symbol Device:R
- removed R11, R13, R15, R17: 91K, Seattle_Synths:R_Axial_DIN0207_L6.3mm_D2.5mm_P10.16mm_Horizontal, symbol Device:R
- removed R12, R14, R16, R18, R8, R9: 100K, Seattle_Synths:R_Axial_DIN0207_L6.3mm_D2.5mm_P10.16mm_Horizontal, symbol Device:R
- removed R2: 72K, Seattle_Synths:R_Axial_DIN0207_L6.3mm_D2.5mm_P10.16mm_Horizontal, symbol Device:R
- removed R20: 51K, Seattle_Synths:R_Axial_DIN0207_L6.3mm_D2.5mm_P10.16mm_Horizontal, symbol Device:R
- removed R3, R7: 50K, Seattle_Synths:R_Axial_DIN0207_L6.3mm_D2.5mm_P10.16mm_Horizontal, symbol Device:R
- removed R4, R5, R6: 220K, Seattle_Synths:R_Axial_DIN0207_L6.3mm_D2.5mm_P10.16mm_Horizontal, symbol Device:R
- removed RV1, RV2: 100K, Seattle_Synths:Potentiometer_Alpha_RD901F-40-00D_Single_Vertical, symbol Device:R_Potentiometer
- removed TP1: RES_CTRL, Seattle_Synths:TestPoint_Pad_4.0x4.0mm, symbol Connector:TestPoint
- removed TP2: +12V, Seattle_Synths:TestPoint_Pad_4.0x4.0mm, symbol Connector:TestPoint
- removed TP3: -12V, Seattle_Synths:TestPoint_Pad_4.0x4.0mm, symbol Connector:TestPoint
- removed TP4: GND, Seattle_Synths:TestPoint_Pad_4.0x4.0mm, symbol Connector:TestPoint
- removed TP5: FREQ_CTRL, Seattle_Synths:TestPoint_Pad_4.0x4.0mm, symbol Connector:TestPoint
- removed TP6: INPUT, Seattle_Synths:TestPoint_Pad_4.0x4.0mm, symbol Connector:TestPoint
- removed TP7: OUTPUT, Seattle_Synths:TestPoint_Pad_4.0x4.0mm, symbol Connector:TestPoint
- added 220pF1: C, symbol Device:C
- added C10, C8: 470nF, Seattle_Synths:CP_Radial_D5.0mm_P2.50mm, symbol Device:C
- added C2, C6: 1µF, symbol Seattle_Synths:C_Polarized
- added C5: 220pF, symbol Device:C
- added C9: 100nF, Seattle_Synths:CP_Radial_D5.0mm_P2.50mm, symbol Device:C
- added C?: 22pF, symbol Device:C
- added J1: AUDIO3_INPUT, symbol Seattle_Synths:AudioJack2_SwitchT
- added J2: AUDIO2_INPUT, symbol Seattle_Synths:AudioJack2_SwitchT
- added J3: AUDIO1_INPUT, symbol Seattle_Synths:AudioJack2_SwitchT
- added J4: RES_INPUT, symbol Seattle_Synths:AudioJack2_SwitchT
- added J?: AUDIO_OUTPUT, symbol Seattle_Synths:AudioJack2_SwitchT
- added J?: 1V/OCT_INPUT, symbol Seattle_Synths:AudioJack2_SwitchT
- added J?: CV2_INPUT, symbol Seattle_Synths:AudioJack2_SwitchT
- added R1, R19: 51K, symbol Seattle_Synths:R
- added R10, R14, R15, R8, R?: 91K, symbol Seattle_Synths:R
- added R11, R13, R16, R2, R4, R5, R9, R? (x3): 100K, symbol Seattle_Synths:R
- added R12, R17, R18: 240K, symbol Seattle_Synths:R
- added R20, R? (x2): 1K, symbol Seattle_Synths:R
- added R3, R?: 300K, symbol Seattle_Synths:R
- added R6: 15K, symbol Seattle_Synths:R
- added R7: 36K, symbol Seattle_Synths:R
- added R? (x2): 180K, symbol Seattle_Synths:R
- added R?: 150K, symbol Seattle_Synths:R
- added R?: 1M5, symbol Seattle_Synths:R
- added R?: 56K, symbol Seattle_Synths:R
- added RV1, RV2, RV3: 100K, symbol Seattle_Synths:R_Potentiometer
- added RV4: 1K5, symbol Seattle_Synths:R_Potentiometer_Trim
- added RV?: 100K, symbol Device:R_Potentiometer_Trim
- added RV?: 20K, symbol Device:R_Potentiometer_Trim
- added RV? (x3): 100K lin, symbol Seattle_Synths:R_Potentiometer
- added U2, U? (x3): TL082, symbol Amplifier_Operational:TL082
- C1: value 300pF -> 22pF; footprint Seattle_Synths:C_Disc_D7.5mm_W2.5mm_P5.00mm -> (none)
- C3, C4: value 300pF -> 220pF; footprint Seattle_Synths:C_Disc_D7.5mm_W2.5mm_P5.00mm -> (none)
- C7: value 10µF -> 100nF
- R21: value 330R -> 1K
Connections:
- net +12V: now also C10.1, C9.1, R1.2, RV?.1, RV?.1, U?.8 (V+); no longer C7.2
- net -12V: now also C7.2, C8.2, R12.2, R17.2, R18.2, R20.2, R?.2, RV?.1, U?.4 (V-)
- net GND: now also C3.2, C4.1, 220pF1.1, C10.2, C5.2, C8.1, C9.2, J1.S, J2.S, J3.S, J4.S, J?.S, J?.S, J?.S, R6.2, R?.2, RV1.3, RV2.3, RV3.3, RV?.3, RV?.3, RV?.3, U?.3 (+), U?.5 (+); no longer C1.1, C3.1, C4.2
- net OUT1: now also R10.2, R9.2
- net OUT2: now also R11.2, R15.2
- net OUT3: now also R13.2, R14.2
- net OUT4: now also C6.1, R16.2, R?.2
- net at U1.1 (IN1): now also R8.1, R9.1
- net at U1.11 (CAP4): now also C5.1; no longer C4.1
- net VCFI: now reaches U1.12 (VCFI)
- net VCFI: now also R?.1, R?.2
- net at U1.13 (VEE): now also RV4.3
- net at U1.16 (CAP3): now also C4.2
- net at U1.17 (IN3): now also R13.1, R15.1, R17.1
- net at U1.18 (IN4): now also R14.1, R16.1, R18.1
- net at U1.2 (IN2): now also R10.1, R11.1, R12.1
- net at U1.4 (CAP2): now also C3.1; no longer C1.2
- net at U1.5 (CAP1): now also 220pF1.2; no longer C3.2
- net IRES: now reaches U1.9 (IRES)
- net IRES: now also R2.2
- net VRES: no longer names the net of U1.8 (VRES)
- net VRES: now also R19.2
- new net: C2.1, R8.2
- new net: C1.1, R3.1, R4.1, R5.1, R7.2, U2.2 (-)
- new net: J1.T, R3.2
- new net: R4.2, RV2.2
- new net: J2.T, RV2.1
- new net: R5.2, RV3.2
- new net: J3.T, RV3.1
- new net: C1.2, C2.2, R7.1, U2.1
- new net: R6.1, U2.3 (+)
- new net: C6.2, R19.1
- new net: R20.1, RV4.1, RV4.2
- new net: J4.TN, R1.1
- new net: J4.T, RV1.1
- new net: R2.1, RV1.2
- new net: C?.1, R?.1, R?.2, U?.1
- new net: C?.2, R?.1, R?.1, R?.2, U?.2 (-)
- new net: J?.T, R?.1
- new net: R?.2, RV?.2, RV?.3
- new net: R?.1, R?.1, R?.1, R?.1, R?.1, R?.2, U?.6 (-)
- new net: J?.T, R?.2
- new net: R?.2, RV?.2 (x3)
- new net: R?.1, RV?.1, RV?.2, U?.7
- new net: R?.1, RV?.3
- new net: J?.T, RV?.1
- no-connect marks 4 -> 3
Other:
- moved on the sheet: U1

Commit message: Schematic Rev. 2
Changed lines of the file:
@@
-$Comp
-L Seattle_Synths:R R?
-U 1 1 603A57CE
-P 2400 4150
-F 0 "R?" V 2500 4150 50  0000 C CNN
-F 1 "180K" V 2400 4150 50  0000 C CNN
-F 2 "" V 2330 4150 50  0001 C CNN
-F 3 "~" H 2400 4150 50  0001 C CNN
-	1    2400 4150
-	0    1    -1   0
-$EndComp
 $Comp
 L Seattle_Synths:R R?
@@
 	1    0    0    -1
 $EndComp
-Wire Wire Line
-	2550 3950 2550 4150
-Wire Wire Line
-	2550 4150 2550 4300
-Connection ~ 2550 4150
 Connection ~ 2550 6300
-$Comp
-L power:-12V #PWR?
-U 1 1 603D8FE0
-P 2250 4150
-F 0 "#PWR?" H 2250 4250 50  0001 C CNN
-F 1 "-12V" V 2250 4350 50  0000 C CNN
-F 2 "" H 2250 4150 50  0001 C CNN
-F 3 "" H 2250 4150 50  0001 C CNN
-	1    2250 4150
-	0    -1   -1   0
-$EndComp
 $Comp
 L Seattle_Synths:R R?
@@
 Text Label 4050 5350 0    50   ~ 0
 VCFI
+Connection ~ 2550 4150
+Wire Wire Line
+	2550 4150 2550 4300
+Wire Wire Line
+	2550 3950 2550 4150
+$Comp
+L Seattle_Synths:R R?
+U 1 1 603A57CE
+P 2400 4150
+F 0 "R?" V 2500 4150 50  0000 C CNN
+F 1 "180K" V 2400 4150 50  0000 C CNN
+F 2 "" V 2330 4150 50  0001 C CNN
+F 3 "~" H 2400 4150 50  0001 C CNN
+	1    2400 4150
+	0    1    -1   0
+$EndComp
+$Comp
+L power:-12V #PWR?
+U 1 1 603D8FE0
+P 2100 4150
+F 0 "#PWR?" H 2100 4250 50  0001 C CNN
+F 1 "-12V" V 2100 4350 50  0000 C CNN
+F 2 "" H 2100 4150 50  0001 C CNN
+F 3 "" H 2100 4150 50  0001 C CNN
+	1    2100 4150
+	0    -1   -1   0
+$EndComp
+Wire Wire Line
+	2100 4150 2250 4150
 $EndSCHEMATC

Commit message: Schematic Rev. 2
Parts:
- added unit 3 of U3
- gave numbers to parts that had none: 23
- renumbered C9 to C10, C10 to C11, J5 to J7, R5 to R10, R6 to R12, R7 to R13, R8 to R16, R9 to R17, R10 to R18, R11 to R19, R12 to R20, R13 to R21, R14 to R22, R15 to R23, R16 to R24, R17 to R25, R18 to R26, R19 to R27, R20 to R28, R21 to R29, R3 to R8, R4 to R9, RV2 to RV5, RV3 to RV6, RV4 to RV8, U2 to U1, U1 to U2
Connections:
- net +12V: now also U3.8 (V+)
- net -12V: now also U3.4 (V-)
- no-connect marks 3 -> 6
Other:
- moved on the sheet: C10, C11, C7, C8, C9, D1, J7, J8, R28, R29, R30, R31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

Commit message: Refactor
Parts:
- C1, C3, C4, C5, C9: footprint (none) -> Seattle_Synths:C_0603_1608Metric
- C10, C11, C7, C8: footprint Seattle_Synths:CP_Radial_D5.0mm_P2.50mm -> Seattle_Synths:C_0603_1608Metric
- C12: renamed from 220pF1; value C -> 220pF; footprint (none) -> Seattle_Synths:C_0603_1608Metric
- C2, C6: footprint (none) -> Seattle_Synths:CP_Radial_D5.0mm_P2.50mm
- D1: footprint Seattle_Synths:LED_D5.0mm -> Seattle_Synths:D_0603_1608Metric
- J1, J2, J3, J4, J5, J6, J8: footprint (none) -> Seattle_Synths:Jack_3.5mm_QingPu_WQP-PJ398SM_Vertical_CircularHoles
- J7: footprint Seattle_Synths:PinHeader_2x05_P2.54mm_Vertical -> Seattle_Synths:3M_2510-6002UB
- R1, R10, R11, R12, R13, R14, R15, R16, R17, R18, R19, R2, R20, R21, R22, R23, R24, R25, R26, R27, R28, R3, R30, R31, R32, R33, R4, R5, R6, R7, R8, R9: footprint (none) -> Seattle_Synths:R_0603_1608Metric
- R29: footprint Seattle_Synths:R_Axial_DIN0207_L6.3mm_D2.5mm_P10.16mm_Horizontal -> Seattle_Synths:R_0603_1608Metric
- RV1, RV2, RV3, RV4, RV5, RV6: footprint (none) -> Seattle_Synths:Potentiometer_Alpha_RD901F-40-00D_Single_Vertical
- RV7, RV8, RV9: footprint (none) -> Seattle_Synths:TRIM_3266W-1-102LF
- U1, U3: footprint (none) -> Seattle_Synths:DIP-8_W7.62mm_Socket
